Commit message: testing defining an end effector velocity for g1. Not working at all. Testing on dual_arm.py and works much better

File: Test_Optas/example/robots/g1/meshes/g1_dual_arm copy.urdf (robot description, URDF)
Before this commit: robot g1_dual_arm, 22 links, 21 joints
Links:
- link head_link: geometry collision mesh filename=head_link.STL; visual mesh filename=head_link.STL
- link left_elbow_link: geometry collision mesh filename=left_elbow_link.STL; visual mesh filename=left_elbow_link.STL
- link left_shoulder_pitch_link: geometry collision cylinder length=0.05 radius=0.03; visual mesh filename=left_shoulder_pitch_link.STL
- link left_shoulder_roll_link: geometry collision cylinder length=0.03 radius=0.03; visual mesh filename=left_shoulder_roll_link.STL
- link left_shoulder_yaw_link: geometry collision mesh filename=left_shoulder_yaw_link.STL; visual mesh filename=left_shoulder_yaw_link.STL
- link left_wrist_pitch_link: geometry collision mesh filename=left_wrist_pitch_link.STL; visual mesh filename=left_wrist_pitch_link.STL
- link left_wrist_roll_link: geometry collision mesh filename=left_wrist_roll_link.STL; visual mesh filename=left_wrist_roll_link.STL
- link left_wrist_yaw_link: geometry collision mesh filename=left_wrist_yaw_link.STL; visual mesh filename=left_wrist_yaw_link.STL
- link logo_link: geometry collision mesh filename=logo_link.STL; visual mesh filename=logo_link.STL
- link pelvis: geometry visual mesh filename=pelvis.STL
- link pelvis_contour_link: geometry collision mesh filename=pelvis_contour_link.STL; visual mesh filename=pelvis_contour_link.STL
- link right_elbow_link: geometry collision mesh filename=right_elbow_link.STL; visual mesh filename=right_elbow_link.STL
- link right_shoulder_pitch_link: geometry collision cylinder length=0.05 radius=0.03; visual mesh filename=right_shoulder_pitch_link.STL
- link right_shoulder_roll_link: geometry collision cylinder length=0.03 radius=0.03; visual mesh filename=right_shoulder_roll_link.STL
- link right_shoulder_yaw_link: geometry collision mesh filename=right_shoulder_yaw_link.STL; visual mesh filename=right_shoulder_yaw_link.STL
- link right_wrist_pitch_link: geometry collision mesh filename=right_wrist_pitch_link.STL; visual mesh filename=right_wrist_pitch_link.STL
- link right_wrist_roll_link: geometry collision mesh filename=right_wrist_roll_link.STL; visual mesh filename=right_wrist_roll_link.STL
- link right_wrist_yaw_link: geometry collision mesh filename=right_wrist_yaw_link.STL; visual mesh filename=right_wrist_yaw_link.STL
- link torso_link: geometry collision mesh filename=torso_link.STL; visual mesh filename=torso_link.STL
- link waist_roll_link: geometry visual mesh filename=waist_roll_link.STL
- link waist_support_link: geometry collision mesh filename=waist_support_link.STL; visual mesh filename=waist_support_link.STL
- link waist_yaw_link: geometry visual mesh filename=waist_yaw_link.STL
