Commit message: it throws reasonably well. Sometimes hits the shelf but performs worse when screen recording

File: Test_Optas/example/robots/g1/meshes/g1_dual_arm.urdf (robot description, URDF)
Before this commit: robot g1_29dof_with_hand, 26 links, 26 joints
Links:
- removed link d435_link
- removed link imu_in_pelvis
- removed link imu_in_torso
- removed link mid360_link
Joints:
- removed joint d435_joint
- removed joint imu_in_pelvis_joint
- removed joint imu_in_torso_joint
- removed joint left_hand_palm_joint
- removed joint mid360_joint
- joint left_shoulder_pitch_joint: limit lower=-3.0892 upper=2.6704 effort=25 velocity=37 -> lower=-1.57 upper=2.6704 effort=25 velocity=37
- joint right_shoulder_pitch_joint: limit lower=-3.0892 upper=2.6704 effort=25 velocity=37 -> lower=-1.57 upper=2.6704 effort=25 velocity=37

File: robot/g1/g1_dual_arm.urdf (robot description, URDF)
Before this commit: robot g1_dual_arm, 22 links, 21 joints
Links:
- link head_link: geometry collision mesh filename=meshes/head_link.stl; visual mesh filename=meshes/head_link.stl
- link left_elbow_link: geometry collision mesh filename=meshes/left_elbow_link.stl; visual mesh filename=meshes/left_elbow_link.stl
- link left_shoulder_pitch_link: geometry collision cylinder length=0.05 radius=0.03; visual mesh filename=meshes/left_shoulder_pitch_link.stl
- link left_shoulder_roll_link: geometry collision cylinder length=0.03 radius=0.03; visual mesh filename=meshes/left_shoulder_roll_link.stl
- link left_shoulder_yaw_link: geometry collision mesh filename=meshes/left_shoulder_yaw_link.stl; visual mesh filename=meshes/left_shoulder_yaw_link.stl
- link left_wrist_pitch_link: geometry collision mesh filename=meshes/left_wrist_pitch_link.stl; visual mesh filename=meshes/left_wrist_pitch_link.stl
- link left_wrist_roll_link: geometry collision mesh filename=meshes/left_wrist_roll_link.stl; visual mesh filename=meshes/left_wrist_roll_link.stl
- link left_wrist_yaw_link: geometry collision mesh filename=meshes/left_wrist_yaw_link.stl; visual mesh filename=meshes/left_wrist_yaw_link.stl
- link logo_link: geometry collision mesh filename=meshes/logo_link.stl; visual mesh filename=meshes/logo_link.stl
- link pelvis: geometry visual mesh filename=meshes/pelvis.stl
- link pelvis_contour_link: geometry collision mesh filename=meshes/pelvis_contour_link.stl; visual mesh filename=meshes/pelvis_contour_link.stl
- link right_elbow_link: geometry collision mesh filename=meshes/right_elbow_link.stl; visual mesh filename=meshes/right_elbow_link.stl
- link right_shoulder_pitch_link: geometry collision cylinder length=0.05 radius=0.03; visual mesh filename=meshes/right_shoulder_pitch_link.stl
- link right_shoulder_roll_link: geometry collision cylinder length=0.03 radius=0.03; visual mesh filename=meshes/right_shoulder_roll_link.stl
- link right_shoulder_yaw_link: geometry collision mesh filename=meshes/right_shoulder_yaw_link.stl; visual mesh filename=meshes/right_shoulder_yaw_link.stl
- link right_wrist_pitch_link: geometry collision mesh filename=meshes/right_wrist_pitch_link.stl; visual mesh filename=meshes/right_wrist_pitch_link.stl
- link right_wrist_roll_link: geometry collision mesh filename=meshes/right_wrist_roll_link.stl; visual mesh filename=meshes/right_wrist_roll_link.stl
- link right_wrist_yaw_link: geometry collision mesh filename=meshes/right_wrist_yaw_link.stl; visual mesh filename=meshes/right_wrist_yaw_link.stl
- link torso_link: geometry collision mesh filename=meshes/torso_link.stl; visual mesh filename=meshes/torso_link.stl
- link waist_roll_link: geometry visual mesh filename=meshes/waist_roll_link.stl
- link waist_support_link: geometry collision mesh filename=meshes/waist_support_link.stl; visual mesh filename=meshes/waist_support_link.stl
- link waist_yaw_link: geometry visual mesh filename=meshes/waist_yaw_link.stl
Joints:
- joint waist_pitch_joint: axis 0 1 0 -> (none); limit lower=-0.52 upper=0.52 effort=35 velocity=30 -> (none); type revolute -> fixed
- joint waist_roll_joint: axis 1 0 0 -> (none); limit lower=-0.52 upper=0.52 effort=35 velocity=30 -> (none); type revolute -> fixed

File: robot/g1/meshes/g1_dual_arm.urdf (robot description, URDF)
Before this commit: robot g1_dual_arm, 22 links, 21 joints
Links:
- added link right_hand_base, mass 0.200; collision mesh filename=wristmesh.STL; visual mesh filename=wristmesh.STL
- added link right_hand_thumb_base, mass 0.200; collision mesh filename=FB_palm_ref_MIR.STL; visual mesh filename=FB_palm_ref_MIR.STL
- link head_link: geometry collision mesh filename=head_link.stl; visual mesh filename=head_link.stl
- link left_elbow_link: geometry collision mesh filename=left_elbow_link.stl; visual mesh filename=left_elbow_link.stl
- link left_shoulder_pitch_link: geometry collision cylinder length=0.05 radius=0.03; visual mesh filename=left_shoulder_pitch_link.stl
- link left_shoulder_roll_link: geometry collision cylinder length=0.03 radius=0.03; visual mesh filename=left_shoulder_roll_link.stl
- link left_shoulder_yaw_link: geometry collision mesh filename=left_shoulder_yaw_link.stl; visual mesh filename=left_shoulder_yaw_link.stl
- link left_wrist_pitch_link: geometry collision mesh filename=left_wrist_pitch_link.stl; visual mesh filename=left_wrist_pitch_link.stl
- link left_wrist_roll_link: geometry collision mesh filename=left_wrist_roll_link.stl; visual mesh filename=left_wrist_roll_link.stl
- link left_wrist_yaw_link: geometry collision mesh filename=left_wrist_yaw_link.stl; visual mesh filename=left_wrist_yaw_link.stl
- link logo_link: geometry collision mesh filename=logo_link.stl; visual mesh filename=logo_link.stl
- link pelvis: geometry visual mesh filename=pelvis.stl
- link pelvis_contour_link: geometry collision mesh filename=pelvis_contour_link.stl; visual mesh filename=pelvis_contour_link.stl
- link right_elbow_link: geometry collision mesh filename=right_elbow_link.stl; visual mesh filename=right_elbow_link.stl
- link right_shoulder_pitch_link: geometry collision cylinder length=0.05 radius=0.03; visual mesh filename=right_shoulder_pitch_link.stl
- link right_shoulder_roll_link: geometry collision cylinder length=0.03 radius=0.03; visual mesh filename=right_shoulder_roll_link.stl
- link right_shoulder_yaw_link: geometry collision mesh filename=right_shoulder_yaw_link.stl; visual mesh filename=right_shoulder_yaw_link.stl
- link right_wrist_pitch_link: geometry collision mesh filename=right_wrist_pitch_link.stl; visual mesh filename=right_wrist_pitch_link.stl
- link right_wrist_roll_link: geometry collision mesh filename=right_wrist_roll_link.stl; visual mesh filename=right_wrist_roll_link.stl
- link right_wrist_yaw_link: geometry collision mesh filename=right_wrist_yaw_link.stl; visual mesh filename=right_wrist_yaw_link.stl
- link torso_link: geometry collision mesh filename=torso_link.stl; visual mesh filename=torso_link.stl
- link waist_roll_link: geometry visual mesh filename=waist_roll_link.stl
- link waist_support_link: geometry collision mesh filename=waist_support_link.stl; visual mesh filename=waist_support_link.stl
- link waist_yaw_link: geometry visual mesh filename=waist_yaw_link.stl
Joints:
- added joint g1_wrist_2_hand_base: type fixed, parent right_wrist_yaw_link, child right_hand_base, origin xyz=0.042 0 0 rpy=0 1.57 0
- added joint right_hand_wrist2thumb: type fixed, parent right_hand_base, child right_hand_thumb_base, origin xyz=-24.0476665e-3 3.78124745e-3 32.32964923e-3 rpy=3.14148426 -0.08848813 -3.14036612
- joint left_shoulder_pitch_joint: limit lower=-3.0892 upper=2.6704 effort=25 velocity=37 -> lower=-1.57 upper=2.6704 effort=25 velocity=37
- joint right_shoulder_pitch_joint: limit lower=-3.0892 upper=2.6704 effort=25 velocity=37 -> lower=-1.57 upper=2.6704 effort=25 velocity=37
