Commit message: the throwing mostly works. Hits the shelves but not the clowns

File: robot/g1/g1_dual_arm.urdf (robot description, URDF)
Before this commit: robot g1_dual_arm, 22 links, 21 joints
Links:
- added link center_palm, mass 1.0; collision sphere radius=0.001; visual sphere radius=0.001
- added link right_hand_base, mass 0.200; collision mesh filename=meshes/wristmesh.STL; visual mesh filename=meshes/wristmesh.STL
- added link right_hand_thumb_base, mass 0.200; collision mesh filename=meshes/FB_palm_ref_MIR.STL; visual mesh filename=meshes/FB_palm_ref_MIR.STL
Joints:
- added joint g1_wrist_2_hand_base: type fixed, parent right_wrist_yaw_link, child right_hand_base, origin xyz=0.042 0 0 rpy=0 1.57 0
- added joint hand2ball: type fixed, parent right_hand_base, child center_palm, origin xyz=0.0 -0.002 0.06 rpy=0.349066 0 0
- added joint right_hand_wrist2thumb: type fixed, parent right_hand_base, child right_hand_thumb_base, origin xyz=-24.0476665e-3 3.78124745e-3 32.32964923e-3 rpy=3.14148426 -0.08848813 -3.14036612

File: robot/g1/meshes/ability_hand_left.urdf (robot description, URDF)
Before this commit: robot right_ability_hand, 18 links, 17 joints
Links:
- removed link right_hand_index_anchor
- removed link right_hand_middle_anchor
- removed link right_hand_pinky_anchor
- removed link right_hand_ring_anchor
Joints:
- removed joint right_hand_idx_anchor
- removed joint right_hand_mid_anchor
- removed joint right_hand_pnky_anchor
- removed joint right_hand_rng_anchor
- removed joint right_hand_wrist2thumb
